File: trunk/hardware/usb.sch (KiCad schematic (older format))
At the start: 9 parts, among them J1 USB-MINI-AB, U1 FT232-SSOP28

Commit message: Re-worked power supply boost circuit around an availabel part. Footprint and 3D package added for same.
Fixed multiple DRC errors with default KiCAD parts (saved in local 
library.)

Routed power boost circuit, paying attention to maximum GND/VSS 
shielding.

Set up fills for 50ohm (approx.) traces around radio chip and rest of 
board, both sides.

Updated BOM to reflect latest component changes.
Changed lines of the file:
@@
 LIBS:contrib
 LIBS:valves
-LIBS:freakduino-cache
+LIBS:freakduino-alt-cache
 EELAYER 27 0
 EELAYER END
@@
 $EndComp
 $Comp
-L VSS #PWR030
+L VSS #PWR031
 U 1 1 51E3CBB5
 P 3150 4100
-F 0 "#PWR030" H 3150 4100 30  0001 C CNN
+F 0 "#PWR031" H 3150 4100 30  0001 C CNN
 F 1 "VSS" H 3150 4030 30  0000 C CNN
 F 2 "" H 3150 4100 60  0000 C CNN
@@
 	3150 3300 3150 3050
 $Comp
-L VBUS #PWR031
+L VBUS #PWR032
 U 1 1 51E3CC12
 P 3150 3050
-F 0 "#PWR031" H 3150 3190 20  0001 C CNN
+F 0 "#PWR032" H 3150 3190 20  0001 C CNN
 F 1 "VBUS" H 3150 3160 30  0000 C CNN
 F 2 "" H 3150 3050 60  0000 C CNN
@@
 DP
 $Comp
-L VSS #PWR032
+L VSS #PWR033
 U 1 1 51E3CC1F
 P 5300 5450
-F 0 "#PWR032" H 5300 5450 30  0001 C CNN
+F 0 "#PWR033" H 5300 5450 30  0001 C CNN
 F 1 "VSS" H 5300 5380 30  0000 C CNN
 F 2 "" H 5300 5450 60  0000 C CNN
@@
 Connection ~ 5500 5300
 $Comp
-L VBUS #PWR033
+L VBUS #PWR034
 U 1 1 51E3CC78
 P 5400 2200
-F 0 "#PWR033" H 5400 2340 20  0001 C CNN
+F 0 "#PWR034" H 5400 2340 20  0001 C CNN
 F 1 "VBUS" H 5400 2310 30  0000 C CNN
 F 2 "" H 5400 2200 60  0000 C CNN
@@
 	4200 1950 4200 1750
 $Comp
-L VBUS #PWR034
+L VBUS #PWR035
 U 1 1 51E3CD0B
 P 4200 1750
-F 0 "#PWR034" H 4200 1890 20  0001 C CNN
+F 0 "#PWR035" H 4200 1890 20  0001 C CNN
 F 1 "VBUS" H 4200 1860 30  0000 C CNN
 F 2 "" H 4200 1750 60  0000 C CNN
@@
 $EndComp
 $Comp
-L VSS #PWR035
+L VSS #PWR036
 U 1 1 51E3CD2F
 P 6200 2300
-F 0 "#PWR035" H 6200 2300 30  0001 C CNN
+F 0 "#PWR036" H 6200 2300 30  0001 C CNN
 F 1 "VSS" H 6200 2230 30  0000 C CNN
 F 2 "" H 6200 2300 60  0000 C CNN
@@
 $EndComp
 $Comp
-L VBUS #PWR036
+L VBUS #PWR037
 U 1 1 51E3CD35
 P 6200 1750
-F 0 "#PWR036" H 6200 1890 20  0001 C CNN
+F 0 "#PWR037" H 6200 1890 20  0001 C CNN
 F 1 "VBUS" H 6200 1860 30  0000 C CNN
 F 2 "" H 6200 1750 60  0000 C CNN
@@
 	8400 4000 8400 3700
 $Comp
-L VBUS #PWR037
+L VBUS #PWR038
 U 1 1 51E3CEEA
 P 7900 2450
-F 0 "#PWR037" H 7900 2590 20  0001 C CNN
+F 0 "#PWR038" H 7900 2590 20  0001 C CNN
 F 1 "VBUS" H 7900 2560 30  0000 C CNN
 F 2 "" H 7900 2450 60  0000 C CNN
@@
 $EndComp
 $Comp
-L VBUS #PWR038
+L VBUS #PWR039
 U 1 1 51E3CEF0
 P 8400 2450
-F 0 "#PWR038" H 8400 2590 20  0001 C CNN
+F 0 "#PWR039" H 8400 2590 20  0001 C CNN
 F 1 "VBUS" H 8400 2560 30  0000 C CNN
 F 2 "" H 8400 2450 60  0000 C CNN
@@
 	1    0    0    -1
 $EndComp
-$Comp
-L VSS #PWR039
-U 1 1 51E3D2B6
-P 4150 4750
-F 0 "#PWR039" H 4150 4750 30  0001 C CNN
-F 1 "VSS" H 4150 4680 30  0000 C CNN
-F 2 "" H 4150 4750 60  0000 C CNN
-F 3 "" H 4150 4750 60  0000 C CNN
-	1    4150 4750
-	1    0    0    -1
-$EndComp
-Wire Wire Line
-	4150 4750 4150 4600
-Wire Wire Line
-	4150 4200 4150 4100
-Wire Wire Line
-	4150 4100 4850 4100
 Text Label 4250 4100 0    47   ~ 0
 USB_3V3OUT
@@
 NoConn ~ 6150 4700
 NoConn ~ 6150 4600
+Wire Wire Line
+	4150 4750 4150 4600
+Wire Wire Line
+	4850 4100 4150 4100
+Wire Wire Line
+	4150 4100 4150 4200
+$Comp
+L VSS #PWR041
+U 1 1 51E3D2B6
+P 4150 4750
+F 0 "#PWR041" H 4150 4750 30  0001 C CNN
+F 1 "VSS" H 4150 4680 30  0000 C CNN
+F 2 "" H 4150 4750 60  0000 C CNN
+F 3 "" H 4150 4750 60  0000 C CNN
+	1    4150 4750
+	1    0    0    -1
+$EndComp
 $EndSCHEMATC
